File: airqualitymonitor.kicad_pcb (KiCad board)
At the start: 2 copper layers, 65 x 30.5 mm, 16 parts, among them J1 Conn_SDS011, J2 Conn_01x08, J3 Raspberry_Pi_2_3, U1 BME280, U2 CCS811, U3 CAT24C32

Commit message: Fab proto
Parts:
- J3: moved to B.Cu
- turned J3 to 270 degrees
Routing:
- net GND: track 167.3 -> 214.2 mm
- net /ID_SC: track 13.4 -> 18.9 mm
- net /SDA: track 68.3 -> 64.9 mm
- net +5V: track 58.1 -> 61.0 mm
- net /SCL: track 60.9 -> 58.1 mm
- net /UART_TXD: track 49.9 -> 52.5 mm
- net /CCS811_INTn: track 54.6 -> 52.0 mm
- net /UART_RXD: track 44.9 -> 47.5 mm
- net +3V3: track 103.9 -> 102.1 mm
- net Net-(J3-Pad29): track 0.00 -> 0.70 mm
- net Net-(J3-Pad13): track 0.00 -> 0.70 mm
- added copper zone on B.Cu, net GND

Commit message: Post fab updates
Routing:
- net Net-(R1-Pad2): track 22.8 -> 27.7 mm
- net +3V3: track 102.1 -> 106.5 mm
- net GND: track 214.2 -> 218.3 mm
- net Net-(U2-Pad4): track 0.60 -> 2.69 mm
- net /SDA: track 64.9 -> 66.2 mm
Other:
- board text added: "SDS011"
- board text added: "Temperature Humidity Pressure PM2.5 PM10 VOC CO2"
- board text added: "breathePi"
- board text added: "tokilabs"
- board text added: "tokilabs.co"
